Commit message: Update my_robot.xacro

File: my_robot/urdf/my_robot.xacro (robot description, xacro)
@@ -3,7 +3,7 @@
   <!--Import Plugins-->
   <xacro:include filename="$(find my_robot)/urdf/my_robot.gazebo" />
-  <!--Link (robot_footprint)-->
+  <!--Link: robot_footprint-->
   <link name="robot_footprint"></link>
-  <!--Joint (robot_footprint)-->
+  <!--Joint: robot_footprint & chassis-->
   <joint name="robot_footprint_joint" type="fixed">
     <origin xyz="0 0 0" rpy="0 0 0" />
@@ -11,7 +11,8 @@
     <child link="chassis" />
   </joint>
-  <!--Link (chasiss)-->
+  <!--Link: chasiss-->
   <link name="chassis">
     <pose>0 0 0.1 0 0 0</pose>
+    <!--inertial values-->
     <inertial>
       <mass value="15"/>
@@ -23,4 +24,5 @@
       />
     </inertial>
+    <!--collision values-->
     <collision name="chassis_collision">
       <geometry>
@@ -28,4 +30,5 @@
       </geometry>
     </collision>
+    <!--visual values-->
     <visual name='chassis_visual'>
       <origin rpy="0 0 0" xyz="0 0 0"/>
@@ -34,5 +37,5 @@
       </geometry>
     </visual>
-    <!--front caster-->
+    <!--front caster wheel-->
     <collision name="front_caster_collision">
       <origin xyz="0.35 0 -0.05" rpy=" 0 0 0"/>
@@ -48,9 +51,10 @@
     </visual>
   </link>
-  <!--Link (left_wheel)-->
+  <!--Link: left_wheel-->
   <link name='left_wheel'>
     <inertial>
       <mass value="5"/>
       <origin xyz="0 0 0" rpy="0 1.5707 1.5707" />
+      <!--inertial values-->
       <inertia
           ixx="0.01354166666" ixy="0" ixz="0"
@@ -59,4 +63,5 @@
       />
     </inertial>
+    <!--collision values-->
     <collision name='left_wheel_collision'>
       <origin  xyz="0 0 0" rpy="0 1.5707 1.5707"/>
@@ -65,4 +70,5 @@
       </geometry>
     </collision>
+    <!--visual values-->
     <visual name='left_wheel_visual'>
       <origin xyz="0 0 0" rpy="0 1.5707 1.5707"/>
@@ -72,5 +78,32 @@
     </visual>
   </link>
-  <!--Joint (left_wheel_hinge)-->
+  <!--Link: right_wheel-->
+  <link name="right_wheel">
+    <!--inertial values-->
+    <inertial>
+      <origin xyz="0 0 0" rpy="0 1.5707 1.5707" />
+      <mass value="5"/>
+      <inertia
+          ixx="0.01354166666" ixy="0" ixz="0"
+          iyy="0.01354166666" iyz="0"
+          izz="0.025"
+      />
+    </inertial>
+    <!--collision values-->
+    <collision name="right_wheel_collision">
+      <origin xyz="0 0 0" rpy="0 1.5707 1.5707"/>
+      <geometry>
+        <cylinder length="0.05" radius="0.1"/>
+      </geometry>
+    </collision>
+    <!--visual values-->
+    <visual name="right_wheel_visual">
+      <origin xyz="0 0 0" rpy="0 1.5707 1.5707"/>
+      <geometry>
+        <cylinder length="0.05" radius="0.1"/>
+      </geometry>
+    </visual>
+  </link>
+  <!--Joint: left_wheel_hinge & chassis -->
   <joint name="left_wheel_hinge" type="continuous">
     <origin xyz="-0.05 0.15 0" rpy="0 0 0"/>
@@ -81,29 +114,5 @@
     <joint_properties damping="1.0" friction="1.0" />
   </joint>
-  <!--Link (right_wheel)-->
-  <link name="right_wheel">
-    <inertial>
-      <origin xyz="0 0 0" rpy="0 1.5707 1.5707" />
-      <mass value="5"/>
-      <inertia
-          ixx="0.01354166666" ixy="0" ixz="0"
-          iyy="0.01354166666" iyz="0"
-          izz="0.025"
-      />
-    </inertial>
-    <collision name="right_wheel_collision">
-      <origin xyz="0 0 0" rpy="0 1.5707 1.5707"/>
-      <geometry>
-        <cylinder length="0.05" radius="0.1"/>
-      </geometry>
-    </collision>
-    <visual name="right_wheel_visual">
-      <origin xyz="0 0 0" rpy="0 1.5707 1.5707"/>
-      <geometry>
-        <cylinder length="0.05" radius="0.1"/>
-      </geometry>
-    </visual>
-  </link>
-  <!--Joint (right_wheel_hinge)-->
+  <!--Joint: right_wheel_hinge & chassis -->
   <joint name="right_wheel_hinge" type="continuous">
     <origin xyz="-0.05 -0.15 0" rpy="0 0 0"/>
@@ -114,6 +123,7 @@
     <joint_properties damping="1.0" friction="1.0" />
   </joint>
-  <!--Link (camera)-->
+  <!--Link: camera-->
   <link name='camera'>
+    <!--inertial values-->
     <inertial>
       <origin xyz="0 0 0" rpy="0 0 0"/>
@@ -126,4 +136,5 @@
       />
     </inertial>
+    <!--visual values-->
     <visual name='camera_visual'>
       <origin xyz="0 0 0" rpy="0 0 0"/>
@@ -132,4 +143,5 @@
       </geometry>
     </visual>
+    <!--collision values-->
     <collision name='camera_collision'>
       <origin xyz="0 0 0" rpy="0 0 0"/>
@@ -139,5 +151,5 @@
     </collision>
   </link>
-  <!--Joint (camera)-->
+  <!--Joint: camera-->
   <joint type="fixed" name="camera_joint">
     <origin xyz="0.25 0 0" rpy="0 0 0"/>
@@ -146,6 +158,7 @@
     <axis xyz="0 1 0"/>
   </joint>
-  <!--Links (hokuyo)-->
+  <!--Links: hokuyo lidar -->
   <link name='hokuyo'>
+    <!--inertial values-->
     <inertial>
       <origin xyz="0 0 0" rpy="0 0 0"/>
@@ -157,4 +170,5 @@
       />
     </inertial>
+    <!--visual values-->
     <visual name='hokuyo_visual'>
       <origin xyz="0 0 0" rpy="0 0 0"/>
@@ -163,4 +177,5 @@
       </geometry>
     </visual>
+    <!--collision values-->
     <collision name='hokuyo_collision'>
       <origin xyz="0 0 0" rpy="0 0 0"/>
@@ -170,5 +185,5 @@
     </collision>
   </link>
-  <!--Joint (hokuyo)-->
+  <!--Joint: hokuyo lidar & chassis-->
   <joint type="fixed" name="hokuyo_joint">
     <origin xyz="0.2 0 .07" rpy="0 0 0"/>
@@ -177,19 +192,19 @@
     <axis xyz="0 1 0"/>
   </joint>
-  <!--give your robot some color-->
+  <!--robot colours-->
   <gazebo reference="chassis">
     <material>Gazebo/Yellow</material>
   </gazebo>
   <gazebo reference="left_wheel">
-    <material>Gazebo/Blue</material>
+    <material>Gazebo/Black</material>
   </gazebo>
   <gazebo reference="right_wheel">
-    <material>Gazebo/Blue</material>
+    <material>Gazebo/Black</material>
   </gazebo>
   <gazebo reference="camera">
-    <material>Gazebo/Red</material>
+    <material>Gazebo/Green</material>
   </gazebo>
   <gazebo reference="hokuyo">
-    <material>Gazebo/Black</material>
+    <material>Gazebo/Yellow</material>
   </gazebo>
 </robot>
